File: EMZ/shema/shema.kicad_sch (KiCad schematic)
At the start: 12 parts, among them M1 Motor_DC, M2 Motor_DC, Q1 IRL2505PBF, U1 STM32F030RCTx, U2 SLA7070MPRT, U3 SLA7070MPRT

Commit message: Хардуер верен
Изготвил Веселин Милчев
Parts:
- removed D2: LED, symbol Device:LED
- added D3: LED, symbol Device:LED
Connections:
- net +12V: now also D3.2 (A); no longer Q1.1 (D)
- net GND: now also Q1.3 (S)
- new net: D3.1 (K), Q1.1 (D)
Other:
- moved on the sheet: Q1
Changed lines of the file:
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@@
 	(wire
 		(pts
-			(xy 27.94 161.29) (xy 127 161.29)
+			(xy 27.94 168.91) (xy 127 168.91)
 		)
 		(stroke
@@
 	(wire
 		(pts
-			(xy 27.94 78.74) (xy 27.94 161.29)
+			(xy 27.94 78.74) (xy 27.94 168.91)
 		)
 		(stroke
@@
 	(symbol
 		(lib_id "Simulation_SPICE:NMOS")
-		(at 132.08 161.29 0)
+		(at 132.08 168.91 0)
 		(unit 1)
 		(exclude_from_sim no)
@@
 		(fields_autoplaced yes)
 		(property "Reference" "Q1"
-			(at 138.43 160.0199 0)
+			(at 138.43 167.6399 0)
 			(effects
 				(font
@@
 		)
 		(property "Value" "IRL2505PBF"
-			(at 138.43 162.5599 0)
+			(at 138.43 170.1799 0)
 			(effects
 				(font
@@
 		)
 		(property "Footprint" ""
-			(at 137.16 158.75 0)
+			(at 137.16 166.37 0)
 			(effects
 				(font
@@
 		)
 		(property "Datasheet" "https://ngspice.sourceforge.io/docs/ngspice-html-manual/manual.xhtml#cha_MOSFETs"
-			(at 132.08 173.99 0)
+			(at 132.08 181.61 0)
 			(effects
 				(font
@@
 		)
 		(property "Description" "N-MOSFET transistor, drain/source/gate"
-			(at 132.08 161.29 0)
+			(at 132.08 168.91 0)
 			(effects
 				(font
@@
 		)
 		(property "Sim.Device" "NMOS"
-			(at 132.08 178.435 0)
+			(at 132.08 186.055 0)
 			(effects
 				(font
@@
 		)
 		(property "Sim.Type" "VDMOS"
-			(at 132.08 180.34 0)
+			(at 132.08 187.96 0)
 			(effects
 				(font
@@
 		)
 		(property "Sim.Pins" "1=D 2=G 3=S"
-			(at 132.08 176.53 0)
+			(at 132.08 184.15 0)
 			(effects
 				(font
@@
 				(path "/43583bed-eccb-4d2c-8df6-db17525cdd0e"
 					(reference "Q1")
-					(unit 1)
-				)
-			)
-		)
-	)
-	(symbol
-		(lib_id "power:GND")
-		(at 134.62 173.99 0)
-		(unit 1)
-		(exclude_from_sim no)
-		(in_bom yes)
-		(on_board yes)
-		(dnp no)
-		(fields_autoplaced yes)
-		(property "Reference" "#PWR05"
-			(at 134.62 180.34 0)
-			(effects
-				(font
-					(size 1.27 1.27)
-				)
-				(hide yes)
-			)
-		)
-		(property "Value" "GND"
-			(at 134.62 179.07 0)
-			(effects
-				(font
-					(size 1.27 1.27)
-				)
-			)
-		)
-		(property "Footprint" ""
-			(at 134.62 173.99 0)
-			(effects
-				(font
-					(size 1.27 1.27)
-				)
-				(hide yes)
-			)
-		)
-		(property "Datasheet" ""
-			(at 134.62 173.99 0)
-			(effects
-				(font
-					(size 1.27 1.27)
-				)
-				(hide yes)
-			)
-		)
-		(property "Description" "Power symbol creates a global label with name \"GND\" , ground"
-			(at 134.62 173.99 0)
-			(effects
-				(font
-					(size 1.27 1.27)
-				)
-				(hide yes)
-			)
-		)
-		(pin "1"
-		)
-		(instances
-			(project ""
-				(path "/43583bed-eccb-4d2c-8df6-db17525cdd0e"
-					(reference "#PWR05")
 					(unit 1)
 				)
@@
 	)
 	(symbol
-		(lib_id "Device:LED")
-		(at 134.62 170.18 90)
-		(unit 1)
-		(exclude_from_sim no)
-		(in_bom yes)
-		(on_board yes)
-		(dnp no)
-		(fields_autoplaced yes)
-		(property "Reference" "D2"
-			(at 138.43 170.4974 90)
-			(effects
-				(font
-					(size 1.27 1.27)
-				)
-				(justify right)
-				(hide yes)
-			)
-		)
-		(property "Value" "LED"
-			(at 138.43 173.0374 90)
-			(effects
-				(font
-					(size 1.27 1.27)
-				)
-				(justify right)
-			)
-		)
-		(property "Footprint" ""
-			(at 134.62 170.18 0)
-			(effects
-				(font
-					(size 1.27 1.27)
-				)
-				(hide yes)
-			)
-		)
-		(property "Datasheet" "~"
-			(at 134.62 170.18 0)
-			(effects
-				(font
-					(size 1.27 1.27)
-				)
-				(hide yes)
-			)
-		)
-		(property "Description" "Light emitting diode"
-			(at 134.62 170.18 0)
-			(effects
-				(font
-					(size 1.27 1.27)
-				)
-				(hide yes)
-			)
-		)
-		(property "Sim.Pins" "1=K 2=A"
-			(at 134.62 170.18 0)
-			(effects
-				(font
-					(size 1.27 1.27)
-				)
-				(hide yes)
-			)
-		)
-		(pin "2"
-		)
-		(pin "1"
-		)
-		(instances
-			(project ""
-				(path "/43583bed-eccb-4d2c-8df6-db17525cdd0e"
-					(reference "D2")
-					(unit 1)
-				)
-			)
-		)
-	)
-	(symbol
 		(lib_id "Motor:Motor_DC")
 		(at 171.45 78.74 0)
@@
 				(path "/43583bed-eccb-4d2c-8df6-db17525cdd0e"
 					(reference "M2")
+					(unit 1)
+				)
+			)
+		)
+	)
+	(symbol
+		(lib_id "Device:LED")
+		(at 134.62 160.02 90)
+		(unit 1)
+		(exclude_from_sim no)
+		(in_bom yes)
+		(on_board yes)
+		(dnp no)
+		(fields_autoplaced yes)
+		(property "Reference" "D3"
+			(at 138.43 160.3374 90)
+			(effects
+				(font
+					(size 1.27 1.27)
+				)
+				(justify right)
+				(hide yes)
+			)
+		)
+		(property "Value" "LED"
+			(at 138.43 162.8774 90)
+			(effects
+				(font
+					(size 1.27 1.27)
+				)
+				(justify right)
+			)
+		)
+		(property "Footprint" ""
+			(at 134.62 160.02 0)
+			(effects
+				(font
+					(size 1.27 1.27)
+				)
+				(hide yes)
+			)
+		)
+		(property "Datasheet" "~"
+			(at 134.62 160.02 0)
+			(effects
+				(font
+					(size 1.27 1.27)
+				)
+				(hide yes)
+			)
+		)
+		(property "Description" "Light emitting diode"
+			(at 134.62 160.02 0)
+			(effects
+				(font
+					(size 1.27 1.27)
+				)
+				(hide yes)
+			)
+		)
+		(property "Sim.Pins" "1=K 2=A"
+			(at 134.62 160.02 0)
+			(effects
+				(font
+					(size 1.27 1.27)
+				)
+				(hide yes)
+			)
+		)
+		(pin "2"
+		)
+		(pin "1"
+		)
+		(instances
+			(project "shema"
+				(path "/43583bed-eccb-4d2c-8df6-db17525cdd0e"
+					(reference "D3")
 					(unit 1)
 				)
@@
 					(unit 1)
 				)
+			)
+		)
+	)
+	(symbol
+		(lib_id "power:GND")
+		(at 134.62 173.99 0)
+		(unit 1)
+		(exclude_from_sim no)
+		(in_bom yes)
+		(on_board yes)
+		(dnp no)
+		(fields_autoplaced yes)
+		(property "Reference" "#PWR02"
+			(at 134.62 180.34 0)
+			(effects
+				(font
+					(size 1.27 1.27)
+				)
+				(hide yes)
+			)
+		)
+		(property "Value" "GND"
+			(at 134.62 179.07 0)
+			(effects
+				(font
+					(size 1.27 1.27)
+				)
+			)
+		)
+		(property "Footprint" ""
+			(at 134.62 173.99 0)
+			(effects
+				(font
+					(size 1.27 1.27)
+				)
+				(hide yes)
+			)
+		)
+		(property "Datasheet" ""
+			(at 134.62 173.99 0)
+			(effects
+				(font
+					(size 1.27 1.27)
+				)
+				(hide yes)
+			)
+		)
+		(property "Description" "Power symbol creates a global label with name \"GND\" , ground"
+			(at 134.62 173.99 0)
+			(effects
+				(font
+					(size 1.27 1.27)
+				)
+				(hide yes)
+			)
+		)
+		(pin "1"
+		)
+		(instances
+			(project ""
+				(path "/43583bed-eccb-4d2c-8df6-db17525cdd0e"
+					(reference "#PWR02")
+					(unit 1)
+				)
